File: motordriver.kicad_pcb (KiCad board)
At the start: 2 copper layers, 40.6 x 30.4 mm, 16 parts, among them J1 POWER, M1 Motor_DC, SW1 TASTER_01, SW2 TASTER_02, U1 CD40107BE, U2 L9110

Commit message: initial commit
Parts:
- added REF**: OSHW-Symbol_6.7x6mm_SilkScreen, Symbol:OSHW-Symbol_6.7x6mm_SilkScreen, F.Cu at (147.4, 114.4)
- added REF**: KiCad-Logo2_5mm_SilkScreen, Symbol:KiCad-Logo2_5mm_SilkScreen, F.Cu at (134.0, 114.4)
Other:
- board text added: "JLCJLCJLCJLC"
- board text added: "https://github.com/peddn/motordriver"
